File: Teensy 3.2 reference board clone/T32 ref.sch (EAGLE design)
At the start: 89 parts, among them K1 MK20DX256VLH7, K2 MKL04Z32VLC4, T1 MCP1825S, X1 MINI-USB

Commit message: fix wrong ferrite package
Connections:
- net N$69: now also K1.VOUT33; no longer K1.VOUT3V3
Changed lines of the file:
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@@
 <layer number="94" name="Symbols" color="4" fill="1" visible="yes" active="yes"/>
 <layer number="95" name="Names" color="7" fill="1" visible="yes" active="yes"/>
-<layer number="96" name="Values" color="7" fill="1" visible="no" active="yes"/>
+<layer number="96" name="Values" color="7" fill="1" visible="yes" active="yes"/>
 <layer number="97" name="Info" color="7" fill="1" visible="yes" active="yes"/>
 <layer number="98" name="Guide" color="6" fill="1" visible="yes" active="yes"/>
@@
 <junction x="160.02" y="154.94"/>
 <wire x1="160.02" y1="161.29" x2="160.02" y2="166.37" width="0.1524" layer="91"/>
-<pinref part="K1" gate="G$1" pin="VOUT3V3"/>
+<pinref part="K1" gate="G$1" pin="VOUT33"/>
 <wire x1="109.22" y1="149.86" x2="106.68" y2="149.86" width="0.1524" layer="91"/>
 <wire x1="106.68" y1="149.86" x2="99.06" y2="149.86" width="0.1524" layer="91"/>
